File: pcb/pedal_proto_pcb.kicad_pcb (KiCad board)
At the start: 2 copper layers, 100 x 85 mm, 51 parts, among them J1 GND, J10 RV1_2, J11 RV1_1, J12 RV2_3, J13 RV2_2, J14 RV2_1, J15 RV3_3, J16 RV3_2, J17 RV3_1, J18 RV4_3, J19 RV4_2, J2 GND, J20 RV4_1, J21 stomp_A_1, J22 stomp_A_2, J23 stomp_A_3, J24 stomp_B_1, J25 stomp_B_2, J26 stomp_B_3, J27 stomp_C_1, J28 stomp_C_2, J29 stomp_C_3, J3 GND, J30 switch_1, J31 switch_2, J32 switch_3, J33 GND, J34 VDD, J35 LED-, J36 LED+, J37 GND, J38 input, J39 output, J4 GND, J40 GND, J5 Jack-DC, J6 Barrel_Jack_Output, J7 Barrel_Jack_Input, J8 GND, J9 RV1_3, SW1 SW_3PDT, SW2 SW_SPDT, SW3 SW_SPDT

Commit message: feat: completed pcb
Parts:
- moved R2 37.6 mm to (196.5, 92.5)
- moved D1 5.88 mm to (197.3, 133.0)
- moved R1 5.35 mm to (192.5, 92.5)
- moved J5 3.00 mm to (194.5, 72.0)
- moved D2 2.23 mm to (208.8, 82.0)
Routing:
- net Net-(J34-Pin_1): track 2.54 -> 111.2 mm
- net Net-(J21-Pin_1): track 2.54 -> 95.4 mm
- net Net-(J24-Pin_1): track 2.54 -> 94.3 mm, vias 0 -> 2
- net Net-(J27-Pin_1): track 2.54 -> 87.3 mm
- net Net-(J20-Pin_1): track 2.54 -> 84.4 mm, vias 0 -> 4
- net Net-(J30-Pin_1): track 2.54 -> 84.2 mm
- net Net-(J22-Pin_1): track 3.04 -> 82.3 mm
- net Net-(J25-Pin_1): track 2.54 -> 81.6 mm
- net Net-(J28-Pin_1): track 2.54 -> 76.5 mm
- net Net-(J31-Pin_1): track 2.54 -> 75.4 mm
- net Net-(J39-Pin_1): track 0.00 -> 69.6 mm
- net Net-(J38-Pin_1): track 0.00 -> 69.2 mm
- net Net-(J19-Pin_1): track 2.54 -> 71.2 mm, vias 0 -> 4
- net Net-(J23-Pin_1): track 2.54 -> 66.9 mm
- net Net-(J26-Pin_1): track 2.54 -> 66.8 mm
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Other:
- outline, holes or cut-outs redrawn
- board text added: "FT"
- board text added: "NC"
- board text added: "NO"
